File: chipOne/chipOne_Backup.kicad_pcb (KiCad board)
At the start: 2 copper layers, 25 parts, among them J1 BNC, J2 BNC, U1 Y1247AstimulusGenerator, U10A1 3pinSwitchCustom, U2 Y1247AstimulusGenerator, U3 Y1247AstimulusGenerator, U4 Y1247AstimulusGenerator, U5 CHIP1, U6 3pinSwitchCustom

Commit message: Layout for PCB one made : stage 1
Parts:
- moved C10 32.1 mm to (96.5, 115.0)
- moved C11 32.1 mm to (55.9, 116.9)
- moved C15 32.1 mm to (55.9, 101.0)
- moved C9 32.1 mm to (62.2, 114.8)
- moved U3 32.1 mm to (115.6, 120.7)
- moved U6 32.1 mm to (121.9, 53.3)
- moved C2 32.1 mm to (86.4, 90.2)
- moved C3 32.1 mm to (71.2, 130.8)
- moved C6 32.1 mm to (71.7, 90.2)
- moved C7 32.1 mm to (87.0, 130.8)
- moved J1 32.1 mm to (104.1, 58.4)
- moved J2 32.1 mm to (58.4, 58.4)
- moved U1 32.1 mm to (44.5, 120.7)
- moved U10A1 32.1 mm to (76.2, 53.3)
- moved U4 32.1 mm to (67.3, 74.9)
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Routing:
- net I_clk: track 97.7 -> 50.5 mm, vias 2 -> 1
- net O_outData3: track 71.3 -> 28.9 mm, vias 2 -> 1
- net VDD_core: track 183.5 -> 153.5 mm, vias 8 -> 5
- net I_inData2: track 77.4 -> 48.4 mm, vias 3 -> 1
- net I_DIN: track 55.5 -> 26.6 mm, vias 2 -> 0
- net I_FCLK: track 48.1 -> 27.6 mm, vias 2 -> 0
- net I_reset: track 63.5 -> 44.8 mm, vias 3 -> 1
- net B_outData_bi0: track 62.5 -> 45.3 mm, vias 4 -> 2
- net I_inData3: track 67.5 -> 52.3 mm, vias 5 -> 1
- net O_DOUT: track 49.7 -> 35.5 mm, vias 1 -> 0
- net I_inData1: track 59.6 -> 46.1 mm, vias 5 -> 1
- net B_inData_bi1: track 62.1 -> 49.3 mm, vias 2 -> 1
- net VDD_IO: track 180.9 -> 193.1 mm, vias 6 -> 4
- net B_outData_bi6: track 57.0 -> 46.5 mm, vias 1 -> 2
- net I_testmode: track 49.4 -> 39.0 mm
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- added copper zone on B.Cu, net VSSQ
- added copper zone on F.Cu, net VSSQ
Other:
- board outline added: 116.8 x 106.7 mm
- net class Power: clearance 0.2 -> 0.1; trace_width 0.4 -> 0.8
