File: chipOneTwoCombined/chipOneTwoCombined.kicad_pcb (KiCad board)
At the start: 4 copper layers, 243.2 x 110 mm, 54 parts, among them J1 BNC, J1 Conn_Coaxial, J2 BNC, J2 Conn_Coaxial, J3 5767007-8, J4 5767007-8, U1 Y1247AstimulusGenerator, U10A1 3pinSwitchCustom, U11 3pinSwitchCustom, U2 Y1247AstimulusGenerator, U3 Y1247AstimulusGenerator, U4 Y1247AstimulusGenerator, U5 CHIP1, U5 CHIP2, U6 3pinSwitchCustom

Commit message: Switch changed in both the layout
Parts:
- removed the U6 at (116.8, 63.5)
- removed the U6 at (174.0, 63.5)
- added U6: 3pinSwitchCustom, SW_MS12ANW03:SW_MS12ANW03, F.Cu at (108.1, 59.9)
- added U6: 3pinSwitchCustom, SW_MS12ANW03:SW_MS12ANW03, F.Cu at (167.5, 58.6)
- U10A1, U11: footprint Pin_Headers:Pin_Header_Straight_1x03_Pitch2.54mm -> SW_MS12ANW03:SW_MS12ANW03
- moved U10A1 9.57 mm to (41.8, 60.4), turned to 180 degrees
- moved U11 8.02 mm to (233.8, 58.5), turned to 180 degrees
- moved C16 6.57 mm to (100.5, 89.0)
- moved C7 6.57 mm to (83.9, 119.7)
- moved C12 6.57 mm to (100.5, 104.8)
- moved C13 6.57 mm to (58.3, 89.8)
- moved C11 6.57 mm to (52.2, 105.8)
- moved C15 6.57 mm to (52.2, 89.9)
- moved C9 6.57 mm to (58.3, 105.0)
- moved C2 6.57 mm to (83.2, 79.1)
- moved C3 6.57 mm to (68.8, 119.7)
- moved C6 6.57 mm to (68.5, 78.6)
- moved J3 6.57 mm to (34.5, 134.9)
- moved U2 6.57 mm to (86.4, 133.4)
- moved U3 6.57 mm to (118.3, 109.5)
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Routing:
- net VSSQ: track 769.3 -> 755.0 mm, vias 19 -> 20
- net I_address1: track 147.6 -> 140.2 mm, vias 3 -> 5
- net VDD_IO: track 347.9 -> 352.9 mm
- net VDD_core: track 370.2 -> 373.7 mm
- net VSS_IO: track 781.1 -> 778.5 mm, vias 5 -> 6
- net Net-(J1-Pad1): track 94.4 -> 92.0 mm
- net B_inData_bi7: track 89.8 -> 91.6 mm
- net Net-(J2-Pad1): track 95.1 -> 93.4 mm
- net io[30]: track 151.9 -> 150.4 mm
- net B_outData_bi1: track 69.3 -> 68.3 mm
- net o[5]: track 176.2 -> 175.3 mm
- net B_outData_bi5: track 63.9 -> 64.7 mm
- net I_address5: track 155.1 -> 154.5 mm
Other:
- board size 243.2 x 110 mm -> 245.6 x 110.3 mm

Commit message: Checking for chip two completed, Combined PCB updated
Parts:
- removed C12: 100uF, Capacitors_Tantalum_SMD:CP_Tantalum_Case-X_EIA-7343-43_Hand
- removed C13: 10uF, Capacitors_SMD:C_1206_HandSoldering
- removed J4: 5767007-8, U4164AlogicAnalyser:TE_5767007-8
- removed U3: Y1247AstimulusGenerator, Y1247AstimulusGenerator:ERF8-030-05.0-L-DV-L-TR
- added CPchip2_C12: 100uF, Capacitors_Tantalum_SMD:CP_Tantalum_Case-X_EIA-7343-43_Hand, F.Cu at (193.2, 127.6)
- added CPchip2_C13: 10uF, Capacitors_SMD:C_1206_HandSoldering, F.Cu at (194.8, 78.3)
- added CPchip2_J4: 5767007-8, U4164AlogicAnalyser:TE_5767007-8, F.Cu at (162.0, 137.2)
- added CPchip2_U3: Y1247AstimulusGenerator, Y1247AstimulusGenerator:ERF8-030-05.0-L-DV-L-TR, F.Cu at (191.6, 61.5)
- CPchip1_U5: renamed from U5; value CHIP1 -> CPchip1_CHIP1
- CPchip2_U5: renamed from U5; value CHIP2 -> CPchip2_CHIP2
- moved CPchip2_J3 82.3 mm to (242.3, 137.6)
- moved CPchip1_C16 6.57 mm to (106.7, 91.2)
- moved CPchip1_C7 6.57 mm to (90.1, 121.9)
- moved CPchip1_C12 6.57 mm to (106.7, 107.0)
- moved CPchip1_C13 6.57 mm to (64.5, 92.0)
- moved CPchip1_C11 6.57 mm to (58.4, 108.0)
- moved CPchip1_C15 6.57 mm to (58.4, 92.1)
- moved CPchip1_C9 6.57 mm to (64.5, 107.2)
- moved CPchip1_C2 6.57 mm to (89.4, 81.3)
- moved CPchip1_C3 6.57 mm to (75.0, 121.9)
- moved CPchip1_C6 6.57 mm to (74.7, 80.8)
- moved CPchip1_J3 6.57 mm to (40.6, 137.2)
- moved CPchip1_U2 6.57 mm to (92.6, 135.6)
- moved CPchip1_U3 6.57 mm to (124.5, 111.8)
- moved CPchip1_U5 6.57 mm to (73.5, 94.0)
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- renumbered C1 to CPchip1_C1, C10 to CPchip1_C10, C11 to CPchip1_C11, C12 to CPchip1_C12, C13 to CPchip1_C13, C14 to CPchip1_C14, C15 to CPchip1_C15, C16 to CPchip1_C16, C2 to CPchip1_C2, C3 to CPchip1_C3, C4 to CPchip1_C4, C5 to CPchip1_C5, C6 to CPchip1_C6, C7 to CPchip1_C7, C8 to CPchip1_C8, C9 to CPchip1_C9, J1 to CPchip1_J1, J2 to CPchip1_J2, J3 to CPchip1_J3, J4 to CPchip1_J4, U1 to CPchip1_U1, U10A1 to CPchip1_U10A1, U2 to CPchip1_U2, U3 to CPchip1_U3, U4 to CPchip1_U4, U6 to CPchip1_U6, C1 to CPchip2_C1, C10 to CPchip2_C10, C11 to CPchip2_C11, C14 to CPchip2_C14, C15 to CPchip2_C15, C16 to CPchip2_C16, C2 to CPchip2_C2, C3 to CPchip2_C3, C4 to CPchip2_C4, C5 to CPchip2_C5, C6 to CPchip2_C6, C7 to CPchip2_C7, C8 to CPchip2_C8, C9 to CPchip2_C9, J1 to CPchip2_J1, J2 to CPchip2_J2, J3 to CPchip2_J3, U1 to CPchip2_U1, U11 to CPchip2_U11, U2 to CPchip2_U2, U4 to CPchip2_U4, U6 to CPchip2_U6
Connections:
- CPchip1_J1 pad 1: Net-(J1-Pad1) -> Net-(CPchip1_J1-Pad1)
- CPchip1_J2 pad 1: Net-(J2-Pad1) -> Net-(CPchip1_J2-Pad1)
- CPchip1_J3 pad 1: Net-(J3-Pad1) -> Net-(CPchip1_J3-Pad1)
- CPchip1_J3 pad 2: Net-(J3-Pad2) -> Net-(CPchip1_J3-Pad2)
- CPchip1_J3 pad 3: Net-(J3-Pad3) -> Net-(CPchip1_J3-Pad3)
- CPchip1_J3 pad 4: Net-(J3-Pad4) -> Net-(CPchip1_J3-Pad4)
- CPchip1_U1 pad 1: Net-(U1-Pad1) -> Net-(CPchip1_U1-Pad1)
- CPchip1_U1 pad 10: Net-(U1-Pad10) -> Net-(CPchip1_U1-Pad10)
- CPchip1_U1 pad 11: Net-(U1-Pad11) -> Net-(CPchip1_U1-Pad11)
- CPchip1_U1 pad 12: Net-(U1-Pad12) -> Net-(CPchip1_U1-Pad12)
- CPchip1_U1 pad 13: Net-(U1-Pad13) -> Net-(CPchip1_U1-Pad13)
- CPchip1_U1 pad 14: Net-(U1-Pad14) -> Net-(CPchip1_U1-Pad14)
- CPchip1_U1 pad 15: Net-(U1-Pad15) -> Net-(CPchip1_U1-Pad15)
- CPchip1_U1 pad 16: Net-(U1-Pad16) -> Net-(CPchip1_U1-Pad16)
- CPchip1_U1 pad 17: Net-(U1-Pad17) -> Net-(CPchip1_U1-Pad17)
- CPchip1_U1 pad 18: Net-(U1-Pad18) -> Net-(CPchip1_U1-Pad18)
- CPchip1_U1 pad 19: Net-(U1-Pad19) -> Net-(CPchip1_U1-Pad19)
- CPchip1_U1 pad 2: Net-(U1-Pad2) -> Net-(CPchip1_U1-Pad2)
- CPchip1_U1 pad 20: Net-(U1-Pad20) -> Net-(CPchip1_U1-Pad20)
- CPchip1_U1 pad 22: Net-(U1-Pad22) -> Net-(CPchip1_U1-Pad22)
- CPchip1_U1 pad 3: Net-(U1-Pad3) -> Net-(CPchip1_U1-Pad3)
- CPchip1_U1 pad 37: Net-(U1-Pad37) -> Net-(CPchip1_U1-Pad37)
- CPchip1_U1 pad 4: Net-(U1-Pad4) -> Net-(CPchip1_U1-Pad4)
- CPchip1_U1 pad 40: Net-(U1-Pad40) -> Net-(CPchip1_U1-Pad40)
- CPchip1_U1 pad 41: Net-(U1-Pad41) -> Net-(CPchip1_U1-Pad41)
- CPchip1_U1 pad 44: Net-(U1-Pad44) -> Net-(CPchip1_U1-Pad44)
- CPchip1_U1 pad 5: Net-(U1-Pad5) -> Net-(CPchip1_U1-Pad5)
- CPchip1_U1 pad 6: Net-(U1-Pad6) -> Net-(CPchip1_U1-Pad6)
- CPchip1_U1 pad 7: Net-(U1-Pad7) -> Net-(CPchip1_U1-Pad7)
- CPchip1_U1 pad 8: Net-(U1-Pad8) -> Net-(CPchip1_U1-Pad8)
- CPchip1_U1 pad 9: Net-(U1-Pad9) -> Net-(CPchip1_U1-Pad9)
- CPchip1_U10A1 pad 1: Net-(J2-Pad1) -> Net-(CPchip1_J2-Pad1)
- CPchip1_U2 pad 1: Net-(U2-Pad1) -> Net-(CPchip1_U2-Pad1)
- CPchip1_U2 pad 10: Net-(U2-Pad10) -> Net-(CPchip1_U2-Pad10)
- CPchip1_U2 pad 11: Net-(U2-Pad11) -> Net-(CPchip1_U2-Pad11)
- CPchip1_U2 pad 12: Net-(U2-Pad12) -> Net-(CPchip1_U2-Pad12)
- CPchip1_U2 pad 13: Net-(U2-Pad13) -> Net-(CPchip1_U2-Pad13)
- CPchip1_U2 pad 14: Net-(U2-Pad14) -> Net-(CPchip1_U2-Pad14)
- CPchip1_U2 pad 15: Net-(U2-Pad15) -> Net-(CPchip1_U2-Pad15)
- CPchip1_U2 pad 16: Net-(U2-Pad16) -> Net-(CPchip1_U2-Pad16)
- CPchip1_U2 pad 17: Net-(U2-Pad17) -> Net-(CPchip1_U2-Pad17)
- CPchip1_U2 pad 18: Net-(U2-Pad18) -> Net-(CPchip1_U2-Pad18)
- CPchip1_U2 pad 19: Net-(U2-Pad19) -> Net-(CPchip1_U2-Pad19)
- CPchip1_U2 pad 2: Net-(U2-Pad2) -> Net-(CPchip1_U2-Pad2)
- CPchip1_U2 pad 20: Net-(U2-Pad20) -> Net-(CPchip1_U2-Pad20)
- CPchip1_U2 pad 22: Net-(U2-Pad22) -> Net-(CPchip1_U2-Pad22)
- CPchip1_U2 pad 3: Net-(U2-Pad3) -> Net-(CPchip1_U2-Pad3)
- CPchip1_U2 pad 37: Net-(U2-Pad37) -> Net-(CPchip1_U2-Pad37)
- CPchip1_U2 pad 4: Net-(U2-Pad4) -> Net-(CPchip1_U2-Pad4)
- CPchip1_U2 pad 40: Net-(U2-Pad40) -> Net-(CPchip1_U2-Pad40)
- CPchip1_U2 pad 41: Net-(U2-Pad41) -> Net-(CPchip1_U2-Pad41)
- CPchip1_U2 pad 44: Net-(U2-Pad44) -> Net-(CPchip1_U2-Pad44)
- CPchip1_U2 pad 5: Net-(U2-Pad5) -> Net-(CPchip1_U2-Pad5)
- CPchip1_U2 pad 6: Net-(U2-Pad6) -> Net-(CPchip1_U2-Pad6)
- CPchip1_U2 pad 7: Net-(U2-Pad7) -> Net-(CPchip1_U2-Pad7)
- CPchip1_U2 pad 8: Net-(U2-Pad8) -> Net-(CPchip1_U2-Pad8)
- CPchip1_U2 pad 9: Net-(U2-Pad9) -> Net-(CPchip1_U2-Pad9)
- CPchip1_U4 pad 1: Net-(U4-Pad1) -> Net-(CPchip1_U4-Pad1)
- CPchip1_U4 pad 10: Net-(U4-Pad10) -> Net-(CPchip1_U4-Pad10)
- CPchip1_U4 pad 11: Net-(U4-Pad11) -> Net-(CPchip1_U4-Pad11)
- CPchip1_U4 pad 12: Net-(U4-Pad12) -> Net-(CPchip1_U4-Pad12)
- CPchip1_U4 pad 13: Net-(U4-Pad13) -> Net-(CPchip1_U4-Pad13)
- CPchip1_U4 pad 14: Net-(U4-Pad14) -> Net-(CPchip1_U4-Pad14)
- CPchip1_U4 pad 15: Net-(U4-Pad15) -> Net-(CPchip1_U4-Pad15)
- CPchip1_U4 pad 16: Net-(U4-Pad16) -> Net-(CPchip1_U4-Pad16)
- CPchip1_U4 pad 17: Net-(U4-Pad17) -> Net-(CPchip1_U4-Pad17)
- CPchip1_U4 pad 18: Net-(U4-Pad18) -> Net-(CPchip1_U4-Pad18)
- CPchip1_U4 pad 19: Net-(U4-Pad19) -> Net-(CPchip1_U4-Pad19)
- CPchip1_U4 pad 2: Net-(U4-Pad2) -> Net-(CPchip1_U4-Pad2)
- CPchip1_U4 pad 20: Net-(U4-Pad20) -> Net-(CPchip1_U4-Pad20)
- CPchip1_U4 pad 21: Net-(U4-Pad21) -> Net-(CPchip1_U4-Pad21)
- CPchip1_U4 pad 22: Net-(U4-Pad22) -> Net-(CPchip1_U4-Pad22)
- CPchip1_U4 pad 24: Net-(U4-Pad24) -> Net-(CPchip1_U4-Pad24)
- CPchip1_U4 pad 25: Net-(U4-Pad25) -> Net-(CPchip1_U4-Pad25)
- CPchip1_U4 pad 28: Net-(U4-Pad28) -> Net-(CPchip1_U4-Pad28)
- CPchip1_U4 pad 3: Net-(U4-Pad3) -> Net-(CPchip1_U4-Pad3)
- CPchip1_U4 pad 37: Net-(U4-Pad37) -> Net-(CPchip1_U4-Pad37)
- CPchip1_U4 pad 4: Net-(U4-Pad4) -> Net-(CPchip1_U4-Pad4)
- CPchip1_U4 pad 40: Net-(U4-Pad40) -> Net-(CPchip1_U4-Pad40)
- CPchip1_U4 pad 41: Net-(U4-Pad41) -> Net-(CPchip1_U4-Pad41)
- CPchip1_U4 pad 44: Net-(U4-Pad44) -> Net-(CPchip1_U4-Pad44)
- CPchip1_U4 pad 5: Net-(U4-Pad5) -> Net-(CPchip1_U4-Pad5)
- CPchip1_U4 pad 6: Net-(U4-Pad6) -> Net-(CPchip1_U4-Pad6)
- CPchip1_U4 pad 7: Net-(U4-Pad7) -> Net-(CPchip1_U4-Pad7)
- CPchip1_U4 pad 8: Net-(U4-Pad8) -> Net-(CPchip1_U4-Pad8)
- CPchip1_U4 pad 9: Net-(U4-Pad9) -> Net-(CPchip1_U4-Pad9)
- CPchip1_U6 pad 1: Net-(J1-Pad1) -> Net-(CPchip1_J1-Pad1)
- CPchip2_J1 pad 1: Net-(J1-Pad1) -> Net-(CPchip2_J1-Pad1)
- CPchip2_J2 pad 1: Net-(J2-Pad1) -> Net-(CPchip2_J2-Pad1)
- CPchip2_J3 pad 1: Net-(J3-Pad1) -> Net-(CPchip2_J3-Pad1)
- CPchip2_J3 pad 2: Net-(J3-Pad2) -> Net-(CPchip2_J3-Pad2)
- CPchip2_J3 pad 3: Net-(J3-Pad3) -> Net-(CPchip2_J3-Pad3)
- CPchip2_J3 pad 4: Net-(J3-Pad4) -> Net-(CPchip2_J3-Pad4)
- CPchip2_U1 pad 1: Net-(U1-Pad1) -> Net-(CPchip2_U1-Pad1)
- CPchip2_U1 pad 10: Net-(U1-Pad10) -> Net-(CPchip2_U1-Pad10)
- CPchip2_U1 pad 11: Net-(U1-Pad11) -> Net-(CPchip2_U1-Pad11)
- CPchip2_U1 pad 12: Net-(U1-Pad12) -> Net-(CPchip2_U1-Pad12)
- CPchip2_U1 pad 13: Net-(U1-Pad13) -> Net-(CPchip2_U1-Pad13)
- CPchip2_U1 pad 14: Net-(U1-Pad14) -> Net-(CPchip2_U1-Pad14)
- CPchip2_U1 pad 15: Net-(U1-Pad15) -> Net-(CPchip2_U1-Pad15)
- CPchip2_U1 pad 16: Net-(U1-Pad16) -> Net-(CPchip2_U1-Pad16)
- CPchip2_U1 pad 17: Net-(U1-Pad17) -> Net-(CPchip2_U1-Pad17)
- CPchip2_U1 pad 18: Net-(U1-Pad18) -> Net-(CPchip2_U1-Pad18)
- CPchip2_U1 pad 19: Net-(U1-Pad19) -> Net-(CPchip2_U1-Pad19)
- CPchip2_U1 pad 2: Net-(U1-Pad2) -> Net-(CPchip2_U1-Pad2)
- CPchip2_U1 pad 20: Net-(U1-Pad20) -> Net-(CPchip2_U1-Pad20)
- CPchip2_U1 pad 22: Net-(U1-Pad22) -> Net-(CPchip2_U1-Pad22)
- CPchip2_U1 pad 3: Net-(U1-Pad3) -> Net-(CPchip2_U1-Pad3)
- CPchip2_U1 pad 37: Net-(U1-Pad37) -> Net-(CPchip2_U1-Pad37)
- CPchip2_U1 pad 4: Net-(U1-Pad4) -> Net-(CPchip2_U1-Pad4)
- CPchip2_U1 pad 40: Net-(U1-Pad40) -> Net-(CPchip2_U1-Pad40)
- CPchip2_U1 pad 41: Net-(U1-Pad41) -> Net-(CPchip2_U1-Pad41)
- CPchip2_U1 pad 44: Net-(U1-Pad44) -> Net-(CPchip2_U1-Pad44)
- CPchip2_U1 pad 5: Net-(U1-Pad5) -> Net-(CPchip2_U1-Pad5)
- CPchip2_U1 pad 6: Net-(U1-Pad6) -> Net-(CPchip2_U1-Pad6)
- CPchip2_U1 pad 7: Net-(U1-Pad7) -> Net-(CPchip2_U1-Pad7)
- CPchip2_U1 pad 8: Net-(U1-Pad8) -> Net-(CPchip2_U1-Pad8)
- CPchip2_U1 pad 9: Net-(U1-Pad9) -> Net-(CPchip2_U1-Pad9)
- CPchip2_U11 pad 1: Net-(J2-Pad1) -> Net-(CPchip2_J2-Pad1)
- CPchip2_U2 pad 1: Net-(U2-Pad1) -> Net-(CPchip2_U2-Pad1)
- CPchip2_U2 pad 10: Net-(U2-Pad10) -> Net-(CPchip2_U2-Pad10)
- CPchip2_U2 pad 11: Net-(U2-Pad11) -> Net-(CPchip2_U2-Pad11)
- CPchip2_U2 pad 12: Net-(U2-Pad12) -> Net-(CPchip2_U2-Pad12)
- CPchip2_U2 pad 13: Net-(U2-Pad13) -> Net-(CPchip2_U2-Pad13)
- CPchip2_U2 pad 14: Net-(U2-Pad14) -> Net-(CPchip2_U2-Pad14)
- CPchip2_U2 pad 15: Net-(U2-Pad15) -> Net-(CPchip2_U2-Pad15)
- CPchip2_U2 pad 16: Net-(U2-Pad16) -> Net-(CPchip2_U2-Pad16)
- CPchip2_U2 pad 17: Net-(U2-Pad17) -> Net-(CPchip2_U2-Pad17)
- CPchip2_U2 pad 18: Net-(U2-Pad18) -> Net-(CPchip2_U2-Pad18)
- CPchip2_U2 pad 19: Net-(U2-Pad19) -> Net-(CPchip2_U2-Pad19)
- CPchip2_U2 pad 2: Net-(U2-Pad2) -> Net-(CPchip2_U2-Pad2)
- CPchip2_U2 pad 20: Net-(U2-Pad20) -> Net-(CPchip2_U2-Pad20)
- CPchip2_U2 pad 22: Net-(U2-Pad22) -> Net-(CPchip2_U2-Pad22)
- CPchip2_U2 pad 3: Net-(U2-Pad3) -> Net-(CPchip2_U2-Pad3)
- CPchip2_U2 pad 37: Net-(U2-Pad37) -> Net-(CPchip2_U2-Pad37)
- CPchip2_U2 pad 4: Net-(U2-Pad4) -> Net-(CPchip2_U2-Pad4)
- CPchip2_U2 pad 40: Net-(U2-Pad40) -> Net-(CPchip2_U2-Pad40)
- CPchip2_U2 pad 41: Net-(U2-Pad41) -> Net-(CPchip2_U2-Pad41)
- CPchip2_U2 pad 44: Net-(U2-Pad44) -> Net-(CPchip2_U2-Pad44)
- CPchip2_U2 pad 5: Net-(U2-Pad5) -> Net-(CPchip2_U2-Pad5)
- CPchip2_U2 pad 6: Net-(U2-Pad6) -> Net-(CPchip2_U2-Pad6)
- CPchip2_U2 pad 7: Net-(U2-Pad7) -> Net-(CPchip2_U2-Pad7)
- CPchip2_U2 pad 8: Net-(U2-Pad8) -> Net-(CPchip2_U2-Pad8)
- CPchip2_U2 pad 9: Net-(U2-Pad9) -> Net-(CPchip2_U2-Pad9)
- CPchip2_U4 pad 1: Net-(U4-Pad1) -> Net-(CPchip2_U4-Pad1)
- CPchip2_U4 pad 10: Net-(U4-Pad10) -> Net-(CPchip2_U4-Pad10)
- CPchip2_U4 pad 11: Net-(U4-Pad11) -> Net-(CPchip2_U4-Pad11)
- CPchip2_U4 pad 12: Net-(U4-Pad12) -> Net-(CPchip2_U4-Pad12)
- CPchip2_U4 pad 13: Net-(U4-Pad13) -> Net-(CPchip2_U4-Pad13)
- CPchip2_U4 pad 14: Net-(U4-Pad14) -> Net-(CPchip2_U4-Pad14)
- CPchip2_U4 pad 15: Net-(U4-Pad15) -> Net-(CPchip2_U4-Pad15)
- CPchip2_U4 pad 16: Net-(U4-Pad16) -> Net-(CPchip2_U4-Pad16)
- CPchip2_U4 pad 17: Net-(U4-Pad17) -> Net-(CPchip2_U4-Pad17)
- CPchip2_U4 pad 18: Net-(U4-Pad18) -> Net-(CPchip2_U4-Pad18)
- CPchip2_U4 pad 19: Net-(U4-Pad19) -> Net-(CPchip2_U4-Pad19)
- CPchip2_U4 pad 2: Net-(U4-Pad2) -> Net-(CPchip2_U4-Pad2)
- CPchip2_U4 pad 20: Net-(U4-Pad20) -> Net-(CPchip2_U4-Pad20)
- CPchip2_U4 pad 21: Net-(U4-Pad21) -> Net-(CPchip2_U4-Pad21)
- CPchip2_U4 pad 22: Net-(U4-Pad22) -> Net-(CPchip2_U4-Pad22)
- CPchip2_U4 pad 24: Net-(U4-Pad24) -> Net-(CPchip2_U4-Pad24)
- CPchip2_U4 pad 25: Net-(U4-Pad25) -> Net-(CPchip2_U4-Pad25)
- CPchip2_U4 pad 28: Net-(U4-Pad28) -> Net-(CPchip2_U4-Pad28)
- CPchip2_U4 pad 3: Net-(U4-Pad3) -> Net-(CPchip2_U4-Pad3)
- CPchip2_U4 pad 37: Net-(U4-Pad37) -> Net-(CPchip2_U4-Pad37)
- CPchip2_U4 pad 4: Net-(U4-Pad4) -> Net-(CPchip2_U4-Pad4)
- CPchip2_U4 pad 40: Net-(U4-Pad40) -> Net-(CPchip2_U4-Pad40)
- CPchip2_U4 pad 41: Net-(U4-Pad41) -> Net-(CPchip2_U4-Pad41)
- CPchip2_U4 pad 44: Net-(U4-Pad44) -> Net-(CPchip2_U4-Pad44)
- CPchip2_U4 pad 5: Net-(U4-Pad5) -> Net-(CPchip2_U4-Pad5)
- CPchip2_U4 pad 6: Net-(U4-Pad6) -> Net-(CPchip2_U4-Pad6)
- CPchip2_U4 pad 7: Net-(U4-Pad7) -> Net-(CPchip2_U4-Pad7)
- CPchip2_U4 pad 8: Net-(U4-Pad8) -> Net-(CPchip2_U4-Pad8)
- CPchip2_U4 pad 9: Net-(U4-Pad9) -> Net-(CPchip2_U4-Pad9)
- CPchip2_U6 pad 1: Net-(J1-Pad1) -> Net-(CPchip2_J1-Pad1)
Routing:
- net io[17]: track 180.8 -> 85.2 mm, vias 3 -> 2
- net Net-(J2-Pad1): track 93.4 -> 0.00 mm, vias 2 -> 0
- net Net-(J1-Pad1): track 92.0 -> 0.00 mm, vias 2 -> 0
- net io[9]: track 177.6 -> 87.7 mm, vias 3 -> 2
- net io[14]: track 168.7 -> 83.8 mm, vias 3 -> 2
- net io[11]: track 168.9 -> 89.5 mm, vias 3 -> 2
- net o[5]: track 175.3 -> 96.1 mm, vias 1 -> 2
- net io[12]: track 164.9 -> 86.1 mm, vias 3 -> 0
- net io[16]: track 169.1 -> 90.4 mm, vias 3 -> 1
- net io[8]: track 176.7 -> 98.3 mm
- net io[13]: track 178.4 -> 100.2 mm, vias 3 -> 2
- net io[15]: track 163.3 -> 88.0 mm
- net io[21]: track 190.3 -> 116.5 mm, vias 2 -> 0
- net io[20]: track 172.9 -> 101.5 mm, vias 3 -> 1
- net o[2]: track 159.8 -> 91.4 mm, vias 3 -> 2
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Other:
- board size 245.6 x 110.3 mm -> 241.5 x 110 mm

Commit message: Combined files modified
Parts:
- added CPchip3_C1: 10uF, Capacitors_SMD:C_1206_HandSoldering, B.Cu at (295.7, 132.3)
- added CPchip3_C10: 10uF, Capacitors_SMD:C_1206_HandSoldering, B.Cu at (321.6, 122.2)
- added CPchip3_C11: 100uF, Capacitors_Tantalum_SMD:CP_Tantalum_Case-X_EIA-7343-43_Hand, B.Cu at (279.4, 124.0)
- added CPchip3_C12: 100uF, Capacitors_Tantalum_SMD:CP_Tantalum_Case-X_EIA-7343-43_Hand, B.Cu at (327.7, 123.0)
- added CPchip3_C13: 10uF, Capacitors_SMD:C_1206_HandSoldering, B.Cu at (285.5, 108.0)
- added CPchip3_C14: 10uF, Capacitors_SMD:C_1206_HandSoldering, B.Cu at (321.6, 107.9)
- added CPchip3_C15: 100uF, Capacitors_Tantalum_SMD:CP_Tantalum_Case-X_EIA-7343-43_Hand, B.Cu at (279.4, 108.1)
- added CPchip3_C16: 100uF, Capacitors_Tantalum_SMD:CP_Tantalum_Case-X_EIA-7343-43_Hand, B.Cu at (327.7, 107.2)
- added CPchip3_C2: 10uF, Capacitors_SMD:C_1206_HandSoldering, B.Cu at (310.4, 97.3)
- added CPchip3_C3: 100uF, Capacitors_Tantalum_SMD:CP_Tantalum_Case-X_EIA-7343-43_Hand, B.Cu at (296.0, 137.9)
- added CPchip3_C4: 100uF, Capacitors_Tantalum_SMD:CP_Tantalum_Case-X_EIA-7343-43_Hand, B.Cu at (310.2, 91.7)
- added CPchip3_C5: 10uF, Capacitors_SMD:C_1206_HandSoldering, B.Cu at (310.4, 132.3)
- added CPchip3_C6: 10uF, Capacitors_SMD:C_1206_HandSoldering, B.Cu at (295.7, 96.8)
- added CPchip3_C7: 100uF, Capacitors_Tantalum_SMD:CP_Tantalum_Case-X_EIA-7343-43_Hand, B.Cu at (311.1, 137.9)
- added CPchip3_C8: 100uF, Capacitors_Tantalum_SMD:CP_Tantalum_Case-X_EIA-7343-43_Hand, B.Cu at (294.9, 91.7)
- added CPchip3_C9: 10uF, Capacitors_SMD:C_1206_HandSoldering, B.Cu at (285.5, 123.2)
- added CPchip3_J1: BNC, bnc_connector:TE_227161-1, F.Cu at (335.3, 70.8)
- added CPchip3_J2: BNC, bnc_connector:TE_227161-1, F.Cu at (269.3, 70.6)
- added CPchip3_J3: 5767007-8, U4164AlogicAnalyser:TE_5767007-8, F.Cu at (266.4, 146.4)
- added CPchip3_J4: 5767007-8, U4164AlogicAnalyser:TE_5767007-8, F.Cu at (334.0, 147.0)
- added CPchip3_U1: Y1247AstimulusGenerator, Y1247AstimulusGenerator:ERF8-030-05.0-L-DV-L-TR, F.Cu at (265.0, 126.7)
- added CPchip3_U10A1: 3pinSwitchCustom, SW_MS12ANW03:SW_MS12ANW03, F.Cu at (269.2, 80.8)
- added CPchip3_U2: Y1247AstimulusGenerator, Y1247AstimulusGenerator:ERF8-030-05.0-L-DV-L-TR, F.Cu at (313.0, 153.0)
- added CPchip3_U3: Y1247AstimulusGenerator, Y1247AstimulusGenerator:ERF8-030-05.0-L-DV-L-TR, F.Cu at (346.0, 127.8)
- added CPchip3_U4: Y1247AstimulusGenerator, Y1247AstimulusGenerator:ERF8-030-05.0-L-DV-L-TR, F.Cu at (291.1, 79.5)
- added CPchip3_U5: CPchip3_CHIP1, chip1:280-5205-01, F.Cu at (294.5, 110.0)
- added CPchip3_U6: 3pinSwitchCustom, SW_MS12ANW03:SW_MS12ANW03, F.Cu at (335.3, 81.6)
- moved CPchip2_C1 21.4 mm to (213.3, 126.7)
- moved CPchip2_C10 21.4 mm to (200.7, 96.0)
- moved CPchip2_C11 21.4 mm to (220.3, 126.9)
- moved CPchip2_C12 21.4 mm to (181.7, 145.6)
- moved CPchip2_C13 21.4 mm to (183.3, 96.3)
- moved CPchip2_C14 21.4 mm to (171.2, 123.2)
- moved CPchip2_C16 21.4 mm to (221.0, 109.0)
- moved CPchip2_C2 21.4 mm to (181.8, 137.9)
- moved CPchip2_C3 21.4 mm to (163.6, 107.8)
- moved CPchip2_C4 21.4 mm to (201.0, 89.1)
- moved CPchip2_C5 21.4 mm to (201.5, 138.1)
- moved CPchip2_C6 21.4 mm to (213.2, 108.9)
- moved CPchip2_C7 21.4 mm to (182.9, 89.0)
- moved CPchip2_C8 21.4 mm to (163.6, 124.0)
- moved CPchip2_C9 21.4 mm to (171.0, 107.1)
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Routing:
- net VSSQ: track 759.6 -> 1428.6 mm, vias 20 -> 22
- net VDD_IO: track 352.9 -> 703.9 mm, vias 6 -> 13
- net VDD_core: track 388.5 -> 603.1 mm, vias 10 -> 17
- net I_address3: track 153.5 -> 296.3 mm, vias 5 -> 6
- net I_clk: track 148.5 -> 286.8 mm, vias 4 -> 10
- net I_address0: track 136.8 -> 272.7 mm
- net I_address1: track 140.2 -> 269.0 mm, vias 5 -> 6
- net I_address2: track 135.8 -> 252.6 mm, vias 5 -> 7
- net I_address5: track 150.8 -> 262.7 mm, vias 4 -> 6
- net B_inData_bi0: track 124.0 -> 225.4 mm, vias 3 -> 5
- net B_inData_bi1: track 135.9 -> 237.2 mm, vias 2 -> 3
- net I_inData3: track 103.7 -> 204.9 mm
- net I_address4: track 125.7 -> 226.4 mm, vias 2 -> 3
- net B_outData_bi7: track 153.3 -> 248.8 mm, vias 5 -> 7
- net B_inData_bi6: track 80.8 -> 175.8 mm, vias 3 -> 4
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Other:
- board size 241.5 x 110 mm -> 333 x 109 mm
- net class Default: via_dia 0.4 -> 0.3
- net class Power: via_dia 0.4 -> 0.6; via_drill 0.2 -> 0.4
