File: ChipTwo_newDesign/ChipTwo.sch (KiCad schematic (older format))
At the start: 27 parts

Commit message: A lot of Changes made and the design has been updated
Parts:
- removed CPchip2_J3, CPchip2_J4: 5767007-8, U4164AlogicAnalyser:TE_5767007-8, symbol U4164AlogicAnalyser:5767007-8
- added CPchip2_U10, CPchip2_U9: E5403A_retention, Y1247AstimulusGenerator:E5403A_retention, symbol Y1247AstimulusGenerator:E5403A_retention
Connections:
- wire segments 189 -> 279
- no-connect marks 116 -> 108
