File: chipOne_newDesign/chipOne.sch (KiCad schematic (older format))
At the start: 27 parts

Commit message: A lot of Changes made and the design has been updated
Parts:
- removed CPchip1_J3, CPchip1_J4: 5767007-8, U4164AlogicAnalyser:TE_5767007-8, symbol U4164AlogicAnalyser:5767007-8
- added CPchip1_U10, CPchip1_U9: E5403A_retention, Y1247AstimulusGenerator:E5403A_retention, symbol Y1247AstimulusGenerator:E5403A_retention
Connections:
- no-connect marks 124 -> 116
Other:
- note added: "Logic Analyzer Connectors (E5406A) - Contactless connector"
- note removed: "Logic Analyzer Connectors (U4205)"
